File: V3.1/PowerPCB_mk0.sch (EAGLE design)
At the start: 124 parts, among them CON1 PINHEAD_1X12-2.54-FEMALE, CON2 PINHEAD_1X06-2.54-FEMALE, CON3 PINHEAD_1X02-2.54-FEMALE, CON4 PINHEAD_1X06-2.54-FEMALE, CON7 PINHEAD_1X06-2.54-FEMALE, IC1 TPS54560B, IC10 TPS54260, IC2 TPS54560B, IC3 TPS54560B, IC4 TPS54560B, IC5 INA169, J1 CONNECTION-7MM, M1 BATTERY_CON-XT30-RA, M2 BATTERY_CON-XT30-RA, M3 BATTERY_CON-XT30-RA, M4 BATTERY_CON-XT30-RA, M5 BATTERY_CON-XT30-RA, M6 BATTERY_CON-XT30-RA, M7 BATTERY_CON-XT30-RA, Q1 IRFR2407PBF, Q2 IRFR2407PBF, Q3 IRFR2407PBF

Commit message: InterPCB connectors issues fix
Parts:
- R27: value 143K -> 39K; LCSC# C22877 -> C23153; MANF# 0603WAF1433T5E -> 0603WAF3902T5E
Other:
- note added: "TPS54560/54260 Vout = 0.8 * (Rh/Rl + 1)"
- note added: "Vout = 12,24 V"
- note added: "Vout = 23,68 V"
- note added: "Vout = 3,92 V"
- note added: "Vout = 5.088"
- note removed: "Check this link for PX4 current and voltage sensing setup https://docs.px4.io/v1.12/en/config/battery.html"
- note removed: "Use testpad to check output voltage"
- moved on the sheet: B1H, B1L, B2H, B2L, B3H, B3L, C1, C10, C11, C12, C13, C14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

Commit message: silk updates
Parts:
- added C45: 4700p, rc:C-0603
- C39: value 0.1uF -> 0.1u
- C62: value 10n -> 4700p; ALLOCATED (none) -> +; LCSC# (none) -> C106218; MANF (none) -> YAGEO; MANF# (none) -> CC0603KRX7R9BB472
- R15: LCSC# C23074 -> C22877; MANF# 0603WAF5362T5E -> 0603WAF1433T5E
- R20, R23: value 10K2 -> 10K; LCSC# C22772 -> C160601; MANF UNI-ROYAL(Uniroyal Elec) -> YAGEO; MANF# 0603WAF1022T5E -> RT0603FRD0710KL
Connections:
- net GND: now also C45.2
- net N$20: now also C45.1
Other:
- moved on the sheet: C44, C54

Commit message: Minor fixes here and there
Parts:
- added D11, D12, D13, D6, D7, D8, D9: SMBJ51CA-SMB, TVS_diodes:SMBJ51CA-SMB
- added R26: 700 µOhms, SHUNT_RESISTORS:CURRENT_SHUNT_KELVIN-0.0005R-3920-KELVIN
- added RL: 53K6, rc:R-1%-0603
- R18: value 200 µOhms -> 700 µOhms; device SHUNT_RESISTORS:CURRENT_SHUNT_KELVIN-0.0002R-3920-KELVIN -> SHUNT_RESISTORS:CURRENT_SHUNT_KELVIN-0.0005R-3920-KELVIN; MANF (none) -> TT Electronics; MANF# (none) -> LRMAP3920B-R0007FT; POWER (none) -> 5W; TC (none) -> ±60ppm/°C
- R21: value 82K -> 143K; LCSC# C23254 -> C22877; MANF# 0603WAF8202T5E -> 0603WAF1433T5E
- R22: value 82K -> 18K; LCSC# C23254 -> C25810; MANF UNI-ROYAL(Uniroyal Elec) -> UNI-ROYAL; MANF# 0603WAF8202T5E -> 0603WAF1802T5E
- RL1: value 82K -> DNM; LCSC# C23254 -> C23153; MANF# 0603WAF8202T5E -> 0603WAF3902T5E
- renumbered R19 to RL1
Connections:
- net BATT_CURRENT: now also RL.2
- net GND: now also RL.1
- net N$19: now also R26.S2
- net N$21: now also R26.S1
- net PGND: now also D11.A, D12.A, D13.A, D6.A, D7.A, D8.A, D9.A
- net VBAT: now also D11.C, D12.C, D13.C, D6.C, D7.C, D8.C, D9.C, R26.2
- net VDC: now also R26.1
Other:
- note added: "For most applications, best performance is attained with an RS value that provides a full-scale shunt voltage of 50 mV to 100 mV; maximum input voltage for accurate measurements is 500 mV."
- note added: "Imax = 169 A Vout max = 3.17 V"
- note removed: "L4 may be replaced with SRP1265A-220M from Bourns"
- note removed: "Max differential input voltage for INA169 is 0.5 V"
- moved on the sheet: C40, C45, C62, M1, M2, M3, M4, M5, M6, M7
